File: kiCad_chessLab/_autosave-main_board.kicad_sch (KiCad schematic)
At the start: 0 parts

Commit message: KiCad Libs Config
Other:
- company: (none) -> CampusFab
- title: (none) -> Main Board
Changed lines of the file:
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@@
 	(generator_version "9.0")
 	(paper "A4")
+	(title_block
+		(title "Main Board")
+		(date "2026-03-04")
+		(rev "v1")
+		(company "CampusFab")
+		(comment 1 "By CARP Alexandru")
+	)
 )
