File: kiCad_chessLab/row.kicad_sch (KiCad schematic)
At the start: 2 parts, among them U1 74HC4051

Commit message: Main Board update
Other:
- sheet cell_A1 renamed cell_B1
- sheet cell_A2 renamed cell_B2
- sheet cell_A3 renamed cell_B3
- sheet cell_A4 renamed cell_B4
- sheet cell_A5 renamed cell_B5
- sheet cell_A6 renamed cell_B6
- sheet cell_A7 renamed cell_B7
- sheet cell_A8 renamed cell_B8
Changed lines of the file:
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@@
 			(color 0 0 0 0.0000)
 		)
-		(property "Sheetname" "cell_A6"
+		(property "Sheetname" "cell_B6"
 			(at 117.856 154.686 0)
 			(effects
@@
 			(color 0 0 0 0.0000)
 		)
-		(property "Sheetname" "cell_A7"
+		(property "Sheetname" "cell_B7"
 			(at 159.766 154.686 0)
 			(effects
@@
 			(color 0 0 0 0.0000)
 		)
-		(property "Sheetname" "cell_A2"
+		(property "Sheetname" "cell_B2"
 			(at 117.856 119.126 0)
 			(effects
@@
 			(color 0 0 0 0.0000)
 		)
-		(property "Sheetname" "cell_A5"
+		(property "Sheetname" "cell_B5"
 			(at 73.406 154.686 0)
 			(effects
@@
 			(color 0 0 0 0.0000)
 		)
-		(property "Sheetname" "cell_A3"
+		(property "Sheetname" "cell_B3"
 			(at 159.766 119.126 0)
 			(effects
@@
 			(color 0 0 0 0.0000)
 		)
-		(property "Sheetname" "cell_A4"
+		(property "Sheetname" "cell_B4"
 			(at 205.486 119.126 0)
 			(effects
@@
 			(color 0 0 0 0.0000)
 		)
-		(property "Sheetname" "cell_A8"
+		(property "Sheetname" "cell_B8"
 			(at 205.486 154.686 0)
 			(effects
@@
 			(color 0 0 0 0.0000)
 		)
-		(property "Sheetname" "cell_A1"
+		(property "Sheetname" "cell_B1"
 			(at 73.406 119.126 0)
 			(effects

Commit message: Complete Schematics
Parts:
- renumbered C1 to C12, U1 to U4
Changed lines of the file:
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@@
 		(on_board yes)
 		(dnp no)
-		(property "Reference" "C1"
+		(property "Reference" "C12"
 			(at 86.36 75.184 90)
 			(effects
@@
 			(project "kiCad_chessLab"
 				(path "/767acb05-88fd-4294-8dd3-73f8ac75b0d1/879e1270-2f10-48e2-adb9-8c8e9c331030/018d4994-81df-4c87-9da8-f9e39ef9d83a"
-					(reference "C3")
+					(reference "C29")
 					(unit 1)
 				)
 				(path "/767acb05-88fd-4294-8dd3-73f8ac75b0d1/879e1270-2f10-48e2-adb9-8c8e9c331030/296e5808-6ccf-4e34-bf2f-3d81c1c8d62b"
-					(reference "C48")
+					(reference "C65")
 					(unit 1)
 				)
 				(path "/767acb05-88fd-4294-8dd3-73f8ac75b0d1/879e1270-2f10-48e2-adb9-8c8e9c331030/6fe74388-356e-4c1f-9809-4ea3ae688db6"
-					(reference "C1")
+					(reference "C12")
 					(unit 1)
 				)
 				(path "/767acb05-88fd-4294-8dd3-73f8ac75b0d1/879e1270-2f10-48e2-adb9-8c8e9c331030/8f0f9883-379c-48a0-97e8-5dcb9e7b1ee1"
-					(reference "C21")
+					(reference "C38")
 					(unit 1)
 				)
 				(path "/767acb05-88fd-4294-8dd3-73f8ac75b0d1/879e1270-2f10-48e2-adb9-8c8e9c331030/be543d1a-72e7-46a4-9de0-04e30e7feab4"
-					(reference "C57")
+					(reference "C74")
 					(unit 1)
 				)
 				(path "/767acb05-88fd-4294-8dd3-73f8ac75b0d1/879e1270-2f10-48e2-adb9-8c8e9c331030/c76aad1f-644f-4742-a24b-cced56a5d4ba"
-					(reference "C10")
+					(reference "C20")
 					(unit 1)
 				)
 				(path "/767acb05-88fd-4294-8dd3-73f8ac75b0d1/879e1270-2f10-48e2-adb9-8c8e9c331030/e9ec80c7-4989-43c4-95ac-e74dd33e324f"
-					(reference "C30")
+					(reference "C47")
 					(unit 1)
 				)
 				(path "/767acb05-88fd-4294-8dd3-73f8ac75b0d1/879e1270-2f10-48e2-adb9-8c8e9c331030/ebb25a42-7c79-4d72-8665-53705e26eda3"
-					(reference "C39")
+					(reference "C56")
 					(unit 1)
 				)
@@
 		(dnp no)
 		(fields_autoplaced yes)
-		(property "Reference" "U1"
+		(property "Reference" "U4"
 			(at 94.8533 35.56 0)
 			(effects
@@
 			(project "kiCad_chessLab"
 				(path "/767acb05-88fd-4294-8dd3-73f8ac75b0d1/879e1270-2f10-48e2-adb9-8c8e9c331030/018d4994-81df-4c87-9da8-f9e39ef9d83a"
+					(reference "U6")
+					(unit 1)
+				)
+				(path "/767acb05-88fd-4294-8dd3-73f8ac75b0d1/879e1270-2f10-48e2-adb9-8c8e9c331030/296e5808-6ccf-4e34-bf2f-3d81c1c8d62b"
+					(reference "U10")
+					(unit 1)
+				)
+				(path "/767acb05-88fd-4294-8dd3-73f8ac75b0d1/879e1270-2f10-48e2-adb9-8c8e9c331030/6fe74388-356e-4c1f-9809-4ea3ae688db6"
 					(reference "U4")
 					(unit 1)
 				)
-				(path "/767acb05-88fd-4294-8dd3-73f8ac75b0d1/879e1270-2f10-48e2-adb9-8c8e9c331030/296e5808-6ccf-4e34-bf2f-3d81c1c8d62b"
+				(path "/767acb05-88fd-4294-8dd3-73f8ac75b0d1/879e1270-2f10-48e2-adb9-8c8e9c331030/8f0f9883-379c-48a0-97e8-5dcb9e7b1ee1"
+					(reference "U7")
+					(unit 1)
+				)
+				(path "/767acb05-88fd-4294-8dd3-73f8ac75b0d1/879e1270-2f10-48e2-adb9-8c8e9c331030/be543d1a-72e7-46a4-9de0-04e30e7feab4"
+					(reference "U11")
+					(unit 1)
+				)
+				(path "/767acb05-88fd-4294-8dd3-73f8ac75b0d1/879e1270-2f10-48e2-adb9-8c8e9c331030/c76aad1f-644f-4742-a24b-cced56a5d4ba"
+					(reference "U5")
+					(unit 1)
+				)
+				(path "/767acb05-88fd-4294-8dd3-73f8ac75b0d1/879e1270-2f10-48e2-adb9-8c8e9c331030/e9ec80c7-4989-43c4-95ac-e74dd33e324f"
 					(reference "U8")
 					(unit 1)
 				)
-				(path "/767acb05-88fd-4294-8dd3-73f8ac75b0d1/879e1270-2f10-48e2-adb9-8c8e9c331030/6fe74388-356e-4c1f-9809-4ea3ae688db6"
-					(reference "U1")
-					(unit 1)
-				)
-				(path "/767acb05-88fd-4294-8dd3-73f8ac75b0d1/879e1270-2f10-48e2-adb9-8c8e9c331030/8f0f9883-379c-48a0-97e8-5dcb9e7b1ee1"
-					(reference "U5")
-					(unit 1)
-				)
-				(path "/767acb05-88fd-4294-8dd3-73f8ac75b0d1/879e1270-2f10-48e2-adb9-8c8e9c331030/be543d1a-72e7-46a4-9de0-04e30e7feab4"
+				(path "/767acb05-88fd-4294-8dd3-73f8ac75b0d1/879e1270-2f10-48e2-adb9-8c8e9c331030/ebb25a42-7c79-4d72-8665-53705e26eda3"
 					(reference "U9")
 					(unit 1)
 				)
-				(path "/767acb05-88fd-4294-8dd3-73f8ac75b0d1/879e1270-2f10-48e2-adb9-8c8e9c331030/c76aad1f-644f-4742-a24b-cced56a5d4ba"
-					(reference "U3")
-					(unit 1)
-				)
-				(path "/767acb05-88fd-4294-8dd3-73f8ac75b0d1/879e1270-2f10-48e2-adb9-8c8e9c331030/e9ec80c7-4989-43c4-95ac-e74dd33e324f"
-					(reference "U6")
-					(unit 1)
-				)
-				(path "/767acb05-88fd-4294-8dd3-73f8ac75b0d1/879e1270-2f10-48e2-adb9-8c8e9c331030/ebb25a42-7c79-4d72-8665-53705e26eda3"
-					(reference "U7")
-					(unit 1)
-				)

Commit message: PCB SetUp
Parts:
- U4: footprint (none) -> chessLab-footprints:74HC4051D653
Changed lines of the file:
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@@
 			)
 		)
-		(property "Footprint" ""
+		(property "Footprint" "chessLab-footprints:74HC4051D653"
 			(at 92.71 60.96 0)
 			(effects
