File: kiCad_chessLab/cell.kicad_sch (KiCad schematic)
At the start: 5 parts, among them IC2 A3144EUA

Commit message: KiCad Bug Fix
Changed lines of the file:
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@@
 		(color 0 0 0 0)
-	)
-	(bus_entry
-		(at 50.8 77.47)
-		(size 2.54 2.54)
-		(stroke
-			(width 0)
-			(type default)
-		)
 	)
 	(wire

Commit message: Main Board update
Parts:
- removed R1: 33, Resistor_SMD:R_0603_1608Metric_Pad0.98x0.95mm_HandSolder, symbol Device:R
Connections:
- net DIN: now also LED2.4-DIN (DI)

Commit message: Complete Schematics
Parts:
- renumbered C2 to C11, IC2 to IC5, LED2 to LED1, R9 to R18

Commit message: Hall effect Replaced and 3d files uploaded
Parts:
- removed IC5: A3144EUA, A3144EUA, symbol chessLab-symbols:A3144EUA
- added IC5: SS49E, TO130P160X410X300-3P, symbol chessLab-symbols:SS49E
Connections:
- net GND: now also IC5.2 (-)
- net SIG: now also IC5.3 (O)
- net VCC_3V3: now also IC5.1 (+)
Changed lines of the file:
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@@
 	)
 	(symbol
-		(lib_id "chessLab-symbols:A3144EUA")
+		(lib_id "chessLab-symbols:SS49E")
 		(at 137.16 64.77 0)
 		(unit 1)
@@
 		(fields_autoplaced yes)
 		(property "Reference" "IC5"
-			(at 158.75 66.0399 0)
+			(at 153.67 66.0399 0)
 			(effects
 				(font
@@
 			)
 		)
-		(property "Value" "A3144EUA"
-			(at 158.75 68.5799 0)
+		(property "Value" "SS49E"
+			(at 153.67 68.5799 0)
 			(effects
 				(font
@@
 			)
 		)
-		(property "Footprint" "A3144EUA"
-			(at 158.75 159.69 0)
+		(property "Footprint" "TO130P160X410X300-3P"
+			(at 153.67 159.69 0)
 			(effects
 				(font
@@
 			)
 		)
-		(property "Datasheet" "https://pdf1.alldatasheet.com/datasheet-pdf/download/90853/ALLEGRO/A3144EUA.html"
-			(at 158.75 259.69 0)
+		(property "Datasheet" "https://datasheet.datasheetarchive.com/originals/distributors/SFDatasheet-1/sf-00023632.pdf"
+			(at 153.67 259.69 0)
 			(effects
 				(font
@@
 			)
 		)
-		(property "Description" "SENSITIVE HALL-EFFECT SWITCHES FOR HIGH-TEMPERATURE OPERATION"
+		(property "Description" "Honeywell Ratiometric Hall Effect Sensor switching current 1.5 mA supply voltage 2.7  6.5 V dc"
 			(at 137.16 64.77 0)
 			(effects
@@
 			)
 		)
-		(property "Height" "5.26"
-			(at 158.75 459.69 0)
+		(property "Height" "1.6"
+			(at 153.67 459.69 0)
 			(effects
 				(font
@@
 			)
 		)
-		(property "Manufacturer_Name" "Allegro Microsystems"
-			(at 158.75 559.69 0)
+		(property "Mouser Part Number" "785-SS49E"
+			(at 153.67 559.69 0)
 			(effects
 				(font
@@
 			)
 		)
-		(property "Manufacturer_Part_Number" "A3144EUA"
-			(at 158.75 659.69 0)
+		(property "Mouser Price/Stock" "https://www.mouser.co.uk/ProductDetail/Honeywell/SS49E?qs=%2Ffq2y7sSKcJBD3o5K2Vcgg%3D%3D"
+			(at 153.67 659.69 0)
 			(effects
 				(font
@@
 			)
 		)
-		(property "Mouser Part Number" ""
-			(at 158.75 759.69 0)
+		(property "Manufacturer_Name" "Honeywell"
+			(at 153.67 759.69 0)
 			(effects
 				(font
@@
 			)
 		)
-		(property "Mouser Price/Stock" ""
-			(at 158.75 859.69 0)
+		(property "Manufacturer_Part_Number" "SS49E"
+			(at 153.67 859.69 0)
 			(effects
 				(font
@@
 			)
 		)
-		(property "Arrow Part Number" ""
-			(at 158.75 959.69 0)
-			(effects
-				(font
-					(size 1.27 1.27)
-				)
-				(justify left top)
-				(hide yes)
-			)
-		)
-		(property "Arrow Price/Stock" ""
-			(at 158.75 1059.69 0)
-			(effects
-				(font
-					(size 1.27 1.27)
-				)
-				(justify left top)
-				(hide yes)
-			)
+		(pin "1"
 		)
 		(pin "3"
@@
 		(pin "2"
 		)
-		(pin "1"
-		)
 		(instances
-			(project "kiCad_chessLab"
+			(project ""
 				(path "/767acb05-88fd-4294-8dd3-73f8ac75b0d1/879e1270-2f10-48e2-adb9-8c8e9c331030/018d4994-81df-4c87-9da8-f9e39ef9d83a/1d9f8004-cc8c-4cac-9fc2-6162274561e6"
 					(reference "IC24")
