File: kiCad_chessLab/kiCad_chessLab.kicad_pcb (KiCad board)
At the start: 2 copper layers, 240 x 240 mm, 334 parts, among them IC1 MT3608, IC10 A3144EUA, IC11 A3144EUA, IC12 A3144EUA, IC13 A3144EUA, IC14 A3144EUA, IC15 A3144EUA, IC16 A3144EUA, IC17 A3144EUA, IC18 A3144EUA, IC19 A3144EUA, IC2 TP4056, IC20 A3144EUA, IC21 A3144EUA, IC22 A3144EUA, IC23 A3144EUA, IC24 A3144EUA, IC25 A3144EUA, IC26 A3144EUA, IC27 A3144EUA, IC28 A3144EUA, IC29 A3144EUA, IC3 DW01A-G, IC30 A3144EUA, IC31 A3144EUA, IC32 A3144EUA, IC33 A3144EUA, IC34 A3144EUA, IC35 A3144EUA, IC36 A3144EUA, IC37 A3144EUA, IC38 A3144EUA, IC39 A3144EUA, IC4 ESP32-C6-WROOM-1-N8, IC40 A3144EUA, IC41 A3144EUA, IC42 A3144EUA, IC43 A3144EUA, IC44 A3144EUA, IC45 A3144EUA, IC46 A3144EUA, IC47 A3144EUA, IC48 A3144EUA, IC49 A3144EUA, IC5 A3144EUA, IC50 A3144EUA, IC51 A3144EUA, IC52 A3144EUA, IC53 A3144EUA, IC54 A3144EUA, IC55 A3144EUA, IC56 A3144EUA, IC57 A3144EUA, IC58 A3144EUA, IC59 A3144EUA, IC6 A3144EUA, IC60 A3144EUA, IC61 A3144EUA, IC62 A3144EUA, IC63 A3144EUA, IC64 A3144EUA, IC65 A3144EUA, IC66 A3144EUA, IC67 A3144EUA, IC68 A3144EUA, IC7 A3144EUA, IC8 A3144EUA, IC9 A3144EUA, J1 DATA, J2 PWR, J3 AUX, J4 TYPE-C-31-M-12, J5 DATA, J6 PWR, Q1 FS8205A, Q2 AO3401A, SW1 SW_SPST, SW2 RST, SW3 BOOT, U1 BAT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

Commit message: Hall effect Replaced and 3d files uploaded
Parts:
- added H1: MountingHole_Pad, MountingHole:MountingHole_2.2mm_M2_DIN965_Pad, F.Cu at (34.5, 263.9)
- added H2: MountingHole_Pad, MountingHole:MountingHole_2.2mm_M2_DIN965_Pad, F.Cu at (266.4, 263.9)
- added H3: MountingHole_Pad, MountingHole:MountingHole_2.2mm_M2_DIN965_Pad, F.Cu at (266.6, 32.0)
- added H4: MountingHole_Pad, MountingHole:MountingHole_2.2mm_M2_DIN965_Pad, F.Cu at (34.6, 32.1)
- added H5: MountingHole_Pad, MountingHole:MountingHole_2.2mm_M2_DIN965_Pad, F.Cu at (150.5, 148.0)
- added IC10: SS49E, chessLab-footprints:TO130P160X410X300-3P, F.Cu at (-261.5, -20.1)
- added IC11: SS49E, chessLab-footprints:TO130P160X410X300-3P, F.Cu at (-253.8, -20.1)
- added IC12: SS49E, chessLab-footprints:TO130P160X410X300-3P, F.Cu at (-261.5, -14.9)
- added IC13: SS49E, chessLab-footprints:TO130P160X410X300-3P, F.Cu at (-253.8, 5.65)
- added IC14: SS49E, chessLab-footprints:TO130P160X410X300-3P, F.Cu at (-253.8, 15.9)
- added IC15: SS49E, chessLab-footprints:TO130P160X410X300-3P, F.Cu at (-253.8, 21.1)
- added IC16: SS49E, chessLab-footprints:TO130P160X410X300-3P, F.Cu at (-253.8, -4.65)
- added IC17: SS49E, chessLab-footprints:TO130P160X410X300-3P, F.Cu at (-253.8, 0.50)
- added IC18: SS49E, chessLab-footprints:TO130P160X410X300-3P, F.Cu at (-238.6, -4.65)
- added IC19: SS49E, chessLab-footprints:TO130P160X410X300-3P, F.Cu at (-253.8, 10.8)
- added IC20: SS49E, chessLab-footprints:TO130P160X410X300-3P, F.Cu at (-246.2, -4.65)
- added IC21: SS49E, chessLab-footprints:TO130P160X410X300-3P, F.Cu at (-253.8, -25.2)
- added IC22: SS49E, chessLab-footprints:TO130P160X410X300-3P, F.Cu at (-238.6, -25.2)
- added IC23: SS49E, chessLab-footprints:TO130P160X410X300-3P, F.Cu at (-230.9, -25.2)
- added IC24: SS49E, chessLab-footprints:TO130P160X410X300-3P, F.Cu at (-269.1, -25.2)
- added IC25: SS49E, chessLab-footprints:TO130P160X410X300-3P, F.Cu at (-261.5, -25.2)
- added IC26: SS49E, chessLab-footprints:TO130P160X410X300-3P, F.Cu at (-269.1, -20.1)
- added IC27: SS49E, chessLab-footprints:TO130P160X410X300-3P, F.Cu at (-246.2, -25.2)
- added IC28: SS49E, chessLab-footprints:TO130P160X410X300-3P, F.Cu at (-223.2, -25.2)
- added IC29: SS49E, chessLab-footprints:TO130P160X410X300-3P, F.Cu at (-261.5, 5.65)
- added IC30: SS49E, chessLab-footprints:TO130P160X410X300-3P, F.Cu at (-261.5, 15.9)
- added IC31: SS49E, chessLab-footprints:TO130P160X410X300-3P, F.Cu at (-261.5, 21.1)
- added IC32: SS49E, chessLab-footprints:TO130P160X410X300-3P, F.Cu at (-261.5, -4.65)
- added IC33: SS49E, chessLab-footprints:TO130P160X410X300-3P, F.Cu at (-261.5, 0.50)
- added IC34: SS49E, chessLab-footprints:TO130P160X410X300-3P, F.Cu at (-246.2, -14.9)
- added IC35: SS49E, chessLab-footprints:TO130P160X410X300-3P, F.Cu at (-261.5, 10.8)
- added IC36: SS49E, chessLab-footprints:TO130P160X410X300-3P, F.Cu at (-253.8, -14.9)
- added IC37: SS49E, chessLab-footprints:TO130P160X410X300-3P, F.Cu at (-246.2, 0.50)
- added IC38: SS49E, chessLab-footprints:TO130P160X410X300-3P, F.Cu at (-246.2, 10.8)
- added IC39: SS49E, chessLab-footprints:TO130P160X410X300-3P, F.Cu at (-246.2, 15.9)
- added IC40: SS49E, chessLab-footprints:TO130P160X410X300-3P, F.Cu at (-230.9, -4.65)
- added IC41: SS49E, chessLab-footprints:TO130P160X410X300-3P, F.Cu at (-223.2, -4.65)
- added IC42: SS49E, chessLab-footprints:TO130P160X410X300-3P, F.Cu at (-238.6, 0.50)
- added IC43: SS49E, chessLab-footprints:TO130P160X410X300-3P, F.Cu at (-246.2, 5.65)
- added IC44: SS49E, chessLab-footprints:TO130P160X410X300-3P, F.Cu at (-246.2, 21.1)
- added IC45: SS49E, chessLab-footprints:TO130P160X410X300-3P, F.Cu at (-238.6, 5.65)
- added IC46: SS49E, chessLab-footprints:TO130P160X410X300-3P, F.Cu at (-223.2, 5.65)
- added IC47: SS49E, chessLab-footprints:TO130P160X410X300-3P, F.Cu at (-238.6, 10.8)
- added IC48: SS49E, chessLab-footprints:TO130P160X410X300-3P, F.Cu at (-230.9, 0.50)
- added IC49: SS49E, chessLab-footprints:TO130P160X410X300-3P, F.Cu at (-223.2, 0.50)
- added IC5: SS49E, chessLab-footprints:TO130P160X410X300-3P, F.Cu at (-246.2, -20.1)
- added IC50: SS49E, chessLab-footprints:TO130P160X410X300-3P, F.Cu at (-238.6, 21.1)
- added IC51: SS49E, chessLab-footprints:TO130P160X410X300-3P, F.Cu at (-230.9, 5.65)
- added IC52: SS49E, chessLab-footprints:TO130P160X410X300-3P, F.Cu at (-238.6, 15.9)
- added IC53: SS49E, chessLab-footprints:TO130P160X410X300-3P, F.Cu at (-269.1, -4.65)
- added IC54: SS49E, chessLab-footprints:TO130P160X410X300-3P, F.Cu at (-269.1, 5.65)
- added IC55: SS49E, chessLab-footprints:TO130P160X410X300-3P, F.Cu at (-269.1, 10.8)
- added IC56: SS49E, chessLab-footprints:TO130P160X410X300-3P, F.Cu at (-269.1, -14.9)
- added IC57: SS49E, chessLab-footprints:TO130P160X410X300-3P, F.Cu at (-269.1, -9.80)
- added IC58: SS49E, chessLab-footprints:TO130P160X410X300-3P, F.Cu at (-269.1, 21.1)
- added IC59: SS49E, chessLab-footprints:TO130P160X410X300-3P, F.Cu at (-269.1, 0.50)
- added IC6: SS49E, chessLab-footprints:TO130P160X410X300-3P, F.Cu at (-261.5, -9.80)
- added IC60: SS49E, chessLab-footprints:TO130P160X410X300-3P, F.Cu at (-269.1, 15.9)
- added IC61: SS49E, chessLab-footprints:TO130P160X410X300-3P, F.Cu at (-223.2, -14.9)
- added IC62: SS49E, chessLab-footprints:TO130P160X410X300-3P, F.Cu at (-246.2, -9.80)
- added IC63: SS49E, chessLab-footprints:TO130P160X410X300-3P, F.Cu at (-238.6, -9.80)
- added IC64: SS49E, chessLab-footprints:TO130P160X410X300-3P, F.Cu at (-238.6, -14.9)
- added IC65: SS49E, chessLab-footprints:TO130P160X410X300-3P, F.Cu at (-230.9, -14.9)
- added IC66: SS49E, chessLab-footprints:TO130P160X410X300-3P, F.Cu at (-223.2, -9.80)
- added IC67: SS49E, chessLab-footprints:TO130P160X410X300-3P, F.Cu at (-253.8, -9.80)
- added IC68: SS49E, chessLab-footprints:TO130P160X410X300-3P, F.Cu at (-230.9, -9.80)
- added IC7: SS49E, chessLab-footprints:TO130P160X410X300-3P, F.Cu at (-230.9, -20.1)
- added IC8: SS49E, chessLab-footprints:TO130P160X410X300-3P, F.Cu at (-223.2, -20.1)
- added IC9: SS49E, chessLab-footprints:TO130P160X410X300-3P, F.Cu at (-238.6, -20.1)
- added R82: 0, Resistor_SMD:R_0603_1608Metric_Pad0.98x0.95mm_HandSolder, F.Cu at (-45.4, -90.5)
- IC4: moved to B.Cu
- moved U1 573.4 mm to (366.0, 136.5), turned to 90 degrees
- moved IC4 379.3 mm to (150.4, 254.1)
Connections:
- J1 pad 2: GND -> /power_board/BTN_PWR
- Q2 pad 1: GND -> /power_board/BTN_PWR
- R8 pad 1: GND -> /power_board/BTN_PWR
- R9 pad 1: GND -> /power_board/BTN_PWR
- SW1 pad 2: GND -> /power_board/BTN_PWR
- TP9 pad 1: GND -> /power_board/BTN_PWR
Other:
- board size 240 x 240 mm -> 240 x 239.9 mm
- board text added: "A1"
- board text added: "A2"
- board text added: "A3"
- board text added: "A4"
- board text added: "A5"
- board text added: "A6"
- board text added: "A7"
- board text added: "A8"
- board text added: "B1"
- board text added: "B2"
- board text added: "B3"
- board text added: "B4"
- board text added: "B5"
- board text added: "B6"
- board text added: "B7"
- board text added: "B8"
- board text added: "C1"
- board text added: "C2"
- board text added: "C3"
- board text added: "C4"
- board text added: "C5"
- board text added: "C6"
- board text added: "C7"
- board text added: "C8"
- board text added: "D1"
- board text added: "D2"
- board text added: "D3"
- board text added: "D4"
- board text added: "D5"
- board text added: "D6"
- board text added: "D7"
- board text added: "D8"
- board text added: "E1"
- board text added: "E2"
- board text added: "E3"
- board text added: "E4"
- board text added: "E5"
- board text added: "E6"
- board text added: "E7"
- board text added: "E8"
- board text added: "F1"
- board text added: "F2"
- board text added: "F3"
- board text added: "F4"
- board text added: "F5"
- board text added: "F6"
- board text added: "F7"
- board text added: "F8"
- board text added: "G1"
- board text added: "G2"
- board text added: "G3"
- board text added: "G4"
- board text added: "G5"
- board text added: "G6"
- board text added: "G7"
- board text added: "G8"
- board text added: "H1"
- board text added: "H2"
- board text added: "H3"
- board text added: "H4"
- board text added: "H5"
- board text added: "H6"
- board text added: "H7"
- board text added: "H8"

Commit message: Pcb Continued
Parts:
- C10, C9, J4, J6, R10, R12, R15, R16, R17, U3: moved to B.Cu
- moved J5 435.0 mm to (168.4, 263.5)
- moved IC6 399.9 mm to (44.4, 247.7)
- moved C8 396.7 mm to (180.7, 258.8), turned to 180 degrees
- moved U3 383.9 mm to (181.0, 252.4)
- moved J6 377.7 mm to (127.3, 263.5), turned to 180 degrees
- moved IC5 374.7 mm to (43.4, 217.7)
- moved R15 371.3 mm to (165.0, 247.9)
- moved R11 369.0 mm to (166.1, 244.1)
- moved R16 368.2 mm to (166.9, 244.2)
- moved R13 368.0 mm to (151.4, 251.2), turned to 180 degrees
- moved R17 367.7 mm to (166.9, 246.0), turned to 180 degrees
- moved C9 364.8 mm to (133.2, 261.6), turned to 90 degrees
- moved C10 364.3 mm to (135.5, 261.5), turned to 90 degrees
- moved R14 361.6 mm to (151.4, 245.1), turned to 180 degrees
- moved J4 352.9 mm to (102.2, 265.9), turned to 180 degrees
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
Commit message: pcb Continued
Parts:
- R11: moved to B.Cu
- moved IC42 478.9 mm to (165.1, 258.2)
- moved IC37 469.6 mm to (165.0, 227.3)
- moved IC26 461.2 mm to (102.7, 252.7)
- moved IC34 460.7 mm to (129.2, 252.1)
- moved IC29 452.3 mm to (132.6, 227.6)
- moved IC38 450.2 mm to (163.9, 196.6)
- moved IC39 438.4 mm to (165.1, 167.7)
- moved IC21 438.1 mm to (103.7, 227.9)
- moved IC30 433.6 mm to (132.4, 197.2)
- moved IC43 432.1 mm to (165.1, 138.0)
- moved IC31 421.6 mm to (133.3, 169.0)
- moved C48 420.7 mm to (170.8, 220.3)
- moved LED33 420.7 mm to (164.9, 222.8)
- moved R50 420.7 mm to (170.8, 222.9)
- moved IC35 416.1 mm to (134.1, 139.8)
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
Commit message: Update PCB
Parts:
- removed the IC10 at (-65.9, 21.8)
- removed the IC11 at (-52.1, 21.8)
- removed the IC12 at (-93.4, 75.6)
- removed the IC13 at (-30.0, -106.7)
- removed the IC14 at (-30.0, -79.8)
- removed the IC15 at (-30.0, -66.3)
- removed the IC16 at (-38.4, 75.6)
- removed the IC17 at (-38.4, 89.0)
- removed the IC18 at (-30.0, -39.5)
- removed the IC19 at (-30.0, -93.2)
- removed the IC20 at (-30.0, -52.9)
- removed the IC21 at (-30.0, -26.0)
- removed the IC22 at (-77.1, 6.82)
- removed the IC23 at (-63.4, 6.82)
- removed the IC24 at (-65.9, 48.7)
- removed the IC25 at (-52.1, 89.0)
- removed the IC26 at (-35.9, 6.82)
- removed the IC27 at (-200.5, 74.1)
- removed the IC28 at (-49.6, 6.82)
- removed the IC29 at (-52.1, 35.3)
- removed the IC30 at (-79.6, 48.7)
- removed the IC31 at (-79.6, 62.1)
- removed the IC32 at (-79.6, 35.3)
- removed the IC33 at (-65.9, 35.3)
- removed the IC34 at (-79.6, 89.0)
- removed the IC35 at (-38.4, 35.3)
- removed the IC36 at (-79.6, 75.6)
- removed the IC37 at (-228.0, 74.1)
- removed the IC38 at (-214.3, 60.7)
- removed the IC39 at (-214.3, 74.1)
- removed the IC40 at (-30.0, -12.6)
- removed the IC41 at (-228.0, 60.7)
- removed the IC42 at (-200.5, 60.7)
- removed the IC43 at (-228.0, 87.6)
- removed the IC44 at (-214.3, 87.6)
- removed the IC45 at (-186.8, 74.1)
- removed the IC46 at (-173.0, 60.7)
- removed the IC47 at (-173.0, 74.1)
- removed the IC48 at (-200.5, 87.6)
- removed the IC49 at (-186.8, 60.7)
- removed the IC5 at (-38.4, 21.8)
- removed the IC50 at (-159.3, 60.7)
- removed the IC51 at (-186.8, 87.6)
- removed the IC52 at (-173.0, 87.6)
- removed the IC53 at (-107.1, 48.7)
- removed the IC54 at (-107.1, 75.6)
- removed the IC55 at (-107.1, 89.0)
- removed the IC56 at (-107.1, 21.8)
- removed the IC57 at (-107.1, 35.3)
- removed the IC58 at (-79.6, 21.8)
- removed the IC59 at (-107.1, 62.1)
- removed the IC6 at (-56.6, 169.0)
- removed the IC60 at (-93.4, 21.8)
- removed the IC61 at (-65.9, 62.1)
- removed the IC62 at (-65.9, 89.0)
- removed the IC63 at (-52.1, 62.1)
- removed the IC64 at (-52.1, 48.7)
- removed the IC65 at (-38.4, 48.7)
- removed the IC66 at (-52.1, 75.6)
- removed the IC67 at (-65.9, 75.6)
- removed the IC68 at (-38.4, 62.1)
- removed the IC7 at (-93.4, 48.7)
- removed the IC8 at (-93.4, 62.1)
- removed the IC9 at (-93.4, 35.3)
- moved IC66 548.2 mm to (254.4, 259.3)
- moved IC58 546.2 mm to (222.8, 258.4)
- moved IC53 545.0 mm to (223.8, 227.7)
- moved IC62 541.2 mm to (253.4, 198.4)
- moved IC61 535.4 mm to (254.1, 227.5)
- moved IC54 529.5 mm to (223.6, 199.3)
- moved IC67 528.9 mm to (253.9, 138.1)
- moved IC63 522.3 mm to (252.0, 169.5)
- moved IC55 517.3 mm to (223.4, 168.8)
- moved IC59 511.2 mm to (223.2, 138.0)
- moved IC56 507.3 mm to (223.1, 107.5)
- moved IC64 506.6 mm to (253.4, 105.9)
- moved IC57 501.1 mm to (224.3, 77.4)
- moved IC65 494.0 mm to (253.8, 80.3)
- moved IC60 493.6 mm to (223.5, 46.0)
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Connections:
- IC4 pad 16: /Main Board/A_OUT -> /Main Board/A0
- IC4 pad 26: /Main Board/A0 -> /Main Board/A_OUT

Commit message: Placement
Parts:
- C12, U4: moved to B.Cu
- moved C12 47.5 mm to (54.6, 230.5)
- moved U4 38.4 mm to (56.7, 237.6), turned to -90 degrees
- moved R20 16.2 mm to (44.9, 183.8)
- moved IC29 16.0 mm to (132.6, 211.6)
- moved IC14 15.8 mm to (74.3, 183.6)
- moved IC54 15.6 mm to (224.2, 183.6)
- moved IC62 15.2 mm to (254.2, 183.2)
- moved R31 14.8 mm to (75.2, 245.4)
- moved IC22 14.6 mm to (104.0, 182.8)
- moved IC38 14.5 mm to (164.1, 182.1)
- moved IC45 14.4 mm to (191.6, 212.9)
- moved IC30 14.3 mm to (134.3, 183.0)
- moved IC13 14.0 mm to (74.7, 212.6)
- moved IC21 13.8 mm to (104.1, 214.1)
- moved IC53 13.8 mm to (224.0, 213.9)
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
Commit message: asaa
Parts:
- C8, J5: moved to B.Cu
- R10, R12: moved to F.Cu
- moved IC32 15.1 mm to (140.3, 98.8)
- moved IC17 13.9 mm to (80.1, 68.8)
- moved IC33 13.9 mm to (140.1, 69.1)
- moved IC63 13.7 mm to (260.4, 158.7)
- moved IC15 13.2 mm to (80.4, 158.8)
- moved IC28 13.1 mm to (110.0, 38.8)
- moved IC65 12.9 mm to (259.9, 69.0)
- moved IC36 12.8 mm to (139.8, 38.5)
- moved IC35 12.8 mm to (140.6, 128.8)
- moved IC23 12.6 mm to (110.5, 158.8)
- moved IC20 12.5 mm to (80.1, 38.5)
- moved IC24 12.4 mm to (110.1, 98.7)
- moved IC31 12.4 mm to (140.3, 158.8)
- moved IC55 12.3 mm to (230.4, 158.7)
- moved IC68 12.2 mm to (260.3, 39.1)
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Connections:
- net /Main Board/GPIO12 renamed /Main Board/DN
- net /Main Board/GPIO13 renamed /Main Board/DP
Routing:
- net VBUS: track 0.00 -> 7.11 mm
- net GND: track 0.00 -> 2.73 mm

Commit message: update pcb
Parts:
- C20, C29, C38, C47, C56, C65, C74, R10, R12, U10, U11, U5, U6, U7, U8, U9: moved to B.Cu
- R11: moved to F.Cu
- moved C47 72.7 mm to (173.9, 223.9)
- moved C38 69.6 mm to (143.7, 224.2)
- moved C65 61.2 mm to (232.9, 231.4)
- moved C56 60.2 mm to (202.9, 231.2)
- moved U8 58.9 mm to (176.1, 231.0), turned to -90 degrees
- moved U7 56.0 mm to (145.8, 231.1), turned to -90 degrees
- moved C29 52.7 mm to (114.0, 230.6)
- moved U10 47.6 mm to (235.2, 238.4), turned to -90 degrees
- moved C20 47.2 mm to (85.9, 230.8)
- moved U9 46.7 mm to (205.3, 238.1), turned to -90 degrees
- moved U11 46.6 mm to (264.0, 238.2), turned to -90 degrees
- moved U6 46.4 mm to (116.1, 237.8), turned to -90 degrees
- moved U5 41.0 mm to (85.9, 237.6), turned to -90 degrees
- moved R10 30.9 mm to (130.3, 256.1)
- moved R12 26.7 mm to (124.4, 256.3)
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Routing:
- net +5V: track 0.00 -> 2432.4 mm
- net +3V3: track 0.00 -> 611.6 mm, vias 0 -> 3
- net /Main Board/S2: track 0.00 -> 247.6 mm
- net /Main Board/S0: track 0.00 -> 244.8 mm, vias 0 -> 2
- net /Main Board/S1: track 0.00 -> 238.7 mm, vias 0 -> 2
- net /Main Board/Row_E/DOUT: track 0.00 -> 234.0 mm
- net /Main Board/Row_G/DOUT: track 0.00 -> 233.8 mm
- net /Main Board/Row_C/DOUT: track 0.00 -> 233.4 mm
- net /Main Board/Row_B/DOUT: track 0.00 -> 233.2 mm
- net /Main Board/Row_F/DOUT: track 0.00 -> 232.2 mm
- net /Main Board/Row_D/DOUT: track 0.00 -> 231.9 mm
- net /Main Board/Row_A/DOUT: track 0.00 -> 230.8 mm
- net /Main Board/Row_A/cell_B8/SIG: track 0.00 -> 214.1 mm, vias 0 -> 3
- net /Main Board/Row_A/cell_B7/SIG: track 0.00 -> 169.5 mm, vias 0 -> 1
- net /Main Board/Row_A/En: track 0.00 -> 169.0 mm, vias 0 -> 4
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
Commit message: maj pcb
Parts:
- moved C29 1.94 mm to (115.9, 230.7)
- moved C20 1.75 mm to (84.2, 230.5)
Routing:
- net +3V3: track 611.6 -> 1910.1 mm, vias 3 -> 26
- net GND: track 19.0 -> 254.3 mm, vias 0 -> 22
- net /Main Board/Row_B/cell_B8/SIG: track 0.00 -> 212.8 mm
- net /Main Board/Row_C/cell_B8/SIG: track 0.00 -> 209.6 mm, vias 0 -> 2
- net /Main Board/Row_D/cell_B8/SIG: track 0.00 -> 205.4 mm
- net /Main Board/Row_B/cell_B7/SIG: track 0.00 -> 184.4 mm
- net /Main Board/Row_C/cell_B7/SIG: track 0.00 -> 178.0 mm
- net /Main Board/A_OUT: track 0.00 -> 171.0 mm, vias 0 -> 9
- net /Main Board/Row_D/cell_B7/SIG: track 0.00 -> 165.0 mm
- net /Main Board/Row_C/cell_B6/SIG: track 0.00 -> 150.7 mm
- net /Main Board/Row_B/cell_B6/SIG: track 0.00 -> 150.2 mm
- net /Main Board/Row_D/cell_B6/SIG: track 0.00 -> 138.4 mm, vias 0 -> 2
- net /Main Board/Row_B/En: track 9.58 -> 143.4 mm, vias 1 -> 4
- net /Main Board/Row_C/cell_B5/SIG: track 0.00 -> 109.4 mm
- net /Main Board/Row_B/cell_B5/SIG: track 0.00 -> 108.8 mm
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