File: kiCad_chessLab/kiCad_chessLab.kicad_pcb (KiCad board)
At the start: 2 copper layers, 240 x 239.9 mm, 340 parts, among them IC1 MT3608, IC10 SS49E, IC11 SS49E, IC12 SS49E, IC13 SS49E, IC14 SS49E, IC15 SS49E, IC16 SS49E, IC17 SS49E, IC18 SS49E, IC19 SS49E, IC2 TP4056, IC20 SS49E, IC21 SS49E, IC22 SS49E, IC23 SS49E, IC24 SS49E, IC25 SS49E, IC26 SS49E, IC27 SS49E, IC28 SS49E, IC29 SS49E, IC3 DW01A-G, IC30 SS49E, IC31 SS49E, IC32 SS49E, IC33 SS49E, IC34 SS49E, IC35 SS49E, IC36 SS49E, IC37 SS49E, IC38 SS49E, IC39 SS49E, IC4 ESP32-C6-WROOM-1-N8, IC40 SS49E, IC41 SS49E, IC42 SS49E, IC43 SS49E, IC44 SS49E, IC45 SS49E, IC46 SS49E, IC47 SS49E, IC48 SS49E, IC49 SS49E, IC5 SS49E, IC50 SS49E, IC51 SS49E, IC52 SS49E, IC53 SS49E, IC54 SS49E, IC55 SS49E, IC56 SS49E, IC57 SS49E, IC58 SS49E, IC59 SS49E, IC6 SS49E, IC60 SS49E, IC61 SS49E, IC62 SS49E, IC63 SS49E, IC64 SS49E, IC65 SS49E, IC66 SS49E, IC67 SS49E, IC68 SS49E, IC7 SS49E, IC8 SS49E, IC9 SS49E, J1 DATA, J2 PWR, J3 AUX, J4 TYPE-C-31-M-12, J5 DATA, J6 PWR, Q1 FS8205A, Q2 AO3401A, SW1 SW_SPST, SW2 RST, SW3 BOOT, U1 BAT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

Commit message: maj pcb
Routing:
- net /Main Board/A_OUT: track 171.0 -> 238.6 mm, vias 9 -> 13
- net GND: track 254.3 -> 283.0 mm, vias 22 -> 24
- net /Main Board/Row_E/En: track 0.00 -> 20.5 mm, vias 0 -> 2
- net +3V3: track 1910.1 -> 1930.3 mm, vias 26 -> 29

Commit message: Clean Up Power Board
Parts:
- removed C1, C5: 100uF, Capacitor_SMD:C_1206_3216Metric_Pad1.33x1.80mm_HandSolder
- removed C2, C4, C6, C7: 10uF, Capacitor_SMD:C_0603_1608Metric_Pad1.08x0.95mm_HandSolder
- removed C3: 0.1uF, Capacitor_SMD:C_0603_1608Metric_Pad1.08x0.95mm_HandSolder
- removed D1, D2: CHARGE, LED_SMD:LED_0603_1608Metric_Pad1.05x0.95mm_HandSolder
- removed D3: SS34, Diode_SMD:D_SMA
- removed IC1: MT3608, chessLab-footprints:SOT95P280X145-6N
- removed IC2: TP4056, chessLab-footprints:SOIC127P600X175-9N
- removed IC3: DW01A-G, chessLab-footprints:SOT95P280X135-6N
- removed J1: DATA, Connector_JST:JST_XH_B4B-XH-A_1x04_P2.50mm_Vertical
- removed J2: PWR, Connector_JST:JST_XH_B4B-XH-A_1x04_P2.50mm_Vertical
- removed J3: AUX, Connector_JST:JST_XH_B4B-XH-A_1x04_P2.50mm_Vertical
- removed L1: CDRH4D28NP-2R2NC, chessLab-footprints:CDRH4D28NP100NC
- removed Q1: FS8205A, chessLab-footprints:SOP65P640X120-8N
- removed Q2: AO3401A, Package_TO_SOT_SMD:SOT-23_Handsoldering
- removed R1, R2, R7: 1k, Resistor_SMD:R_0603_1608Metric_Pad0.98x0.95mm_HandSolder
- removed R3: 100, Resistor_SMD:R_0603_1608Metric_Pad0.98x0.95mm_HandSolder
- removed R4: 220k, Resistor_SMD:R_0603_1608Metric_Pad0.98x0.95mm_HandSolder
- removed R5: 33k, Resistor_SMD:R_0603_1608Metric_Pad0.98x0.95mm_HandSolder
- removed R6: 1.1k, Resistor_SMD:R_0603_1608Metric_Pad0.98x0.95mm_HandSolder
- removed R8: 10k, Resistor_SMD:R_0603_1608Metric_Pad0.98x0.95mm_HandSolder
- removed R82: 0, Resistor_SMD:R_0603_1608Metric_Pad0.98x0.95mm_HandSolder
- removed R9: 100k, Resistor_SMD:R_0603_1608Metric_Pad0.98x0.95mm_HandSolder
- removed SW1: SW_SPST, chessLab-footprints:B3U-1000P
- removed TP1: VBUS, TestPoint:TestPoint_Plated_Hole_D2.0mm
- removed TP10: 3V3, TestPoint:TestPoint_Plated_Hole_D2.0mm
- removed TP11, TP13, TP3: GND, TestPoint:TestPoint_Plated_Hole_D2.0mm
- removed TP12: SW_RST, TestPoint:TestPoint_Plated_Hole_D2.0mm
- removed TP2: +BAT, TestPoint:TestPoint_Plated_Hole_D2.0mm
- removed TP4: 5V, TestPoint:TestPoint_Plated_Hole_D2.0mm
- removed TP5: VBAT, TestPoint:TestPoint_Plated_Hole_D2.0mm
- removed TP6: -BAT, TestPoint:TestPoint_Plated_Hole_D2.0mm
- removed TP7: PWR_HOLD, TestPoint:TestPoint_Plated_Hole_D2.0mm
- removed TP8: VSYS, TestPoint:TestPoint_Plated_Hole_D2.0mm
- removed TP9: BTN_PWR, TestPoint:TestPoint_Plated_Hole_D2.0mm
- removed U1: BAT, chessLab-footprints:CONN4_1048_KEY
- removed U2: AMS1117-3.3, Package_TO_SOT_SMD:SOT-223-3_TabPin2
- moved C74 60.3 mm to (261.6, 231.1)
Routing:
- net +3V3: track 1930.3 -> 3010.3 mm, vias 29 -> 59
- net GND: track 283.0 -> 560.7 mm, vias 24 -> 26
- net /Main Board/Row_G/cell_B8/SIG: track 0.00 -> 215.6 mm
- net /Main Board/Row_F/cell_B8/SIG: track 2.50 -> 207.1 mm
- net /Main Board/Row_H/cell_B8/SIG: track 0.00 -> 203.0 mm, vias 0 -> 1
- net /Main Board/Row_E/cell_B8/SIG: track 2.41 -> 201.1 mm
- net /Main Board/Row_G/cell_B7/SIG: track 0.00 -> 183.6 mm
- net /Main Board/Row_H/cell_B7/SIG: track 0.00 -> 172.2 mm
- net /Main Board/Row_F/cell_B7/SIG: track 0.00 -> 171.8 mm
- net /Main Board/Row_E/cell_B7/SIG: track 0.00 -> 167.2 mm
- net /Main Board/Row_H/cell_B6/SIG: track 0.00 -> 150.1 mm
- net /Main Board/Row_G/cell_B6/SIG: track 0.00 -> 147.5 mm
- net /Main Board/Row_F/cell_B6/SIG: track 0.00 -> 147.1 mm, vias 0 -> 2
- net /Main Board/Row_E/cell_B6/SIG: track 0.00 -> 141.7 mm
- net /Main Board/A_OUT: track 238.6 -> 360.8 mm, vias 13 -> 18
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- added copper zone on B.Cu, net GND
- added copper zone on F.Cu, net GND

Commit message: Via stitch
Routing:
- net GND: vias 26 -> 152

Commit message: Final PCB chess
Routing:
- net GND: vias 152 -> 440
