File: kiCad_chessLab/kiCad_chessLab.kicad_sch (KiCad schematic)
At the start: 0 parts

Commit message: Include Lib and readme changes
Other:
- company: (none) -> CampusFab
- title: (none) -> chessLab
Changed lines of the file:
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@@
 	(generator_version "9.0")
 	(paper "A4")
+	(title_block
+		(title "chessLab")
+		(date "2026-03-02")
+		(rev "v1")
+		(company "CampusFab")
+		(comment 1 "By Alexandru Carp")
+	)
 	(sheet_instances
 		(path "/"

Commit message: Svae
Other:
- added sheet Main Board (main_board.kicad_sch)
- added sheet power_board (power_board.kicad_sch)
Changed lines of the file:
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@@
 		(rev "v1")
 		(company "CampusFab")
-		(comment 1 "By Alexandru Carp")
+		(comment 1 "By CARP Alexandru")
+	)
+	(sheet
+		(at 21.59 15.24)
+		(size 234.95 106.68)
+		(exclude_from_sim no)
+		(in_bom yes)
+		(on_board yes)
+		(dnp no)
+		(stroke
+			(width 0.1524)
+			(type solid)
+		)
+		(fill
+			(color 0 0 0 0.0000)
+		)
+		(property "Sheetname" "power_board"
+			(at 21.59 14.5284 0)
+			(effects
+				(font
+					(size 1.27 1.27)
+				)
+				(justify left bottom)
+			)
+		)
+		(property "Sheetfile" "power_board.kicad_sch"
+			(at 21.59 123.698 0)
+			(effects
+				(font
+					(size 1.27 1.27)
+				)
+				(justify left top)
+			)
+		)
+		(instances
+			(project "kiCad_chessLab"
+				(path "/767acb05-88fd-4294-8dd3-73f8ac75b0d1"
+					(page "2")
+				)
+			)
+		)
+	)
+	(sheet
+		(at 22.86 129.54)
+		(size 232.41 29.21)
+		(exclude_from_sim no)
+		(in_bom yes)
+		(on_board yes)
+		(dnp no)
+		(fields_autoplaced yes)
+		(stroke
+			(width 0.1524)
+			(type solid)
+		)
+		(fill
+			(color 0 0 0 0.0000)
+		)
+		(property "Sheetname" "Main Board"
+			(at 22.86 128.8284 0)
+			(effects
+				(font
+					(size 1.27 1.27)
+				)
+				(justify left bottom)
+			)
+		)
+		(property "Sheetfile" "main_board.kicad_sch"
+			(at 22.86 159.3346 0)
+			(effects
+				(font
+					(size 1.27 1.27)
+				)
+				(justify left top)
+			)
+		)
+		(instances
+			(project "kiCad_chessLab"
+				(path "/767acb05-88fd-4294-8dd3-73f8ac75b0d1"
+					(page "3")
+				)
+			)
+		)
 	)
 	(sheet_instances

Commit message: Clean Up Power Board
Other:
- removed sheet power_board
Changed lines of the file:
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@@
-	)
-	(sheet
-		(at 21.59 15.24)
-		(size 234.95 106.68)
-		(exclude_from_sim no)
-		(in_bom yes)
-		(on_board yes)
-		(dnp no)
-		(stroke
-			(width 0.1524)
-			(type solid)
-		)
-		(fill
-			(color 0 0 0 0.0000)
-		)
-		(property "Sheetname" "power_board"
-			(at 21.59 14.5284 0)
-			(effects
-				(font
-					(size 1.27 1.27)
-				)
-				(justify left bottom)
-			)
-		)
-		(property "Sheetfile" "power_board.kicad_sch"
-			(at 21.59 123.698 0)
-			(effects
-				(font
-					(size 1.27 1.27)
-				)
-				(justify left top)
-			)
-		)
-		(instances
-			(project "kiCad_chessLab"
-				(path "/767acb05-88fd-4294-8dd3-73f8ac75b0d1"
-					(page "2")
-				)
-			)
-		)
 	)
 	(sheet
