File: powerBoard/powerBoard.kicad_pcb (KiCad board)
At the start: 2 copper layers, 36 parts, among them J1 DATA, J2 PWR, J3 AUX, Q2 AO3401A, U2 AMS1117-3.3

Commit message: aa
Parts:
- added IC1: MT3608, ChessLab:SOT95P280X145-6N, F.Cu at (140.0, 98.4)
- added IC2: TP4056, ChessLab:SOIC127P600X175-9N, F.Cu at (155.8, 99.5)
- added IC3: DW01A-G, ChessLab:SOT95P280X135-6N, F.Cu at (140.0, 103.0)
- added L1: CDRH4D28NP-2R2NC, ChessLab:CDRH4D28NP100NC, F.Cu at (163.7, 99.8)
- added Q1: FS8205A, ChessLab:SOP65P640X120-8N, F.Cu at (147.1, 98.4)
- added SW1: SW_SPST, ChessLab:B3U-1000P, F.Cu at (170.0, 98.0)
- added U1: BAT, ChessLab:CONN4_1048_KEY, F.Cu at (190.0, 72.0)
- moved J1 33.0 mm to (47.0, 44.2)
- moved J2 33.0 mm to (47.0, 52.0)
- moved J3 33.0 mm to (47.0, 59.8)
- moved U2 33.0 mm to (48.5, 68.4)
Other:
- board outline added: 105 x 85 mm

Commit message: power pcb
Parts:
- removed TP2: +BAT, TestPoint:TestPoint_Plated_Hole_D2.0mm
- removed U1: BAT, ChessLab:CONN4_1048_KEY
- added BAT+1: BAT+, TestPoint:TestPoint_Pad_4.0x4.0mm, F.Cu at (210.0, 97.5)
- added BAT-1: BAT-, TestPoint:TestPoint_Pad_4.0x4.0mm, F.Cu at (203.0, 97.5)
- added H1: MountingHole, MountingHole:MountingHole_2.7mm_M2.5, F.Cu at (144.0, 53.0)
- added H2: MountingHole, MountingHole:MountingHole_2.7mm_M2.5, F.Cu at (238.0, 53.0)
- added H3: MountingHole, MountingHole:MountingHole_2.7mm_M2.5, F.Cu at (238.0, 97.0)
- added H4: MountingHole, MountingHole:MountingHole_2.7mm_M2.5, F.Cu at (144.0, 97.0)
- TP1, TP10, TP13, TP3, TP4, TP5, TP6, TP7, TP8, TP9: footprint TestPoint:TestPoint_Plated_Hole_D2.0mm -> TestPoint:TestPoint_Pad_D2.0mm
- moved U2 183.1 mm to (231.5, 64.0), turned to 90 degrees
- moved J2 169.0 mm to (216.0, 53.0)
- moved J1 148.3 mm to (195.0, 53.0)
- moved C6 147.0 mm to (236.5, 66.5), turned to 90 degrees
- moved R1 144.5 mm to (239.0, 79.0), turned to 180 degrees
- moved R2 144.4 mm to (239.0, 74.0), turned to 180 degrees
- moved C7 140.5 mm to (230.0, 69.5), turned to 180 degrees
- moved C2 137.9 mm to (227.8, 84.6), turned to 180 degrees
- moved C4 137.1 mm to (227.3, 76.6)
- moved R6 136.1 mm to (234.8, 82.6), turned to -90 degrees
- moved D2 135.5 mm to (239.0, 77.0), turned to 180 degrees
- moved D1 135.2 mm to (239.0, 72.0), turned to 180 degrees
- moved J3 127.7 mm to (174.5, 53.0)
- moved R5 115.2 mm to (209.5, 76.0)
- moved R3 115.0 mm to (209.0, 91.0), turned to 180 degrees
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Connections:
- C1 pad 1: /VSYS -> /VBAT
- C6 pad 1: /VSYS -> /VBAT
- IC1 pad 4: /VSYS -> /VBAT
- IC1 pad 5: /VSYS -> /VBAT
- L1 pad 1: /VSYS -> /VBAT
- Q2 pad 3: /VSYS -> /VBAT
- R3 pad 1: Net-(U1-+_1) -> /VBAT
- TP8 pad 1: /VSYS -> /VBAT
- U2 pad 3: /VSYS -> /VBAT
Other:
- board size 105 x 85 mm -> 100 x 50 mm

Commit message: PowerBoard pcb FRev2
Parts:
- removed R82: 0, Resistor_SMD:R_0603_1608Metric_Pad0.98x0.95mm_HandSolder
- removed TP3: GND, TestPoint:TestPoint_Pad_D2.0mm
- removed TP5: VBAT, TestPoint:TestPoint_Pad_D2.0mm
- added JP1: SolderJumper_2_Bridged, Jumper:SolderJumper-2_P1.3mm_Bridged2Bar_Pad1.0x1.5mm, F.Cu at (191.7, 66.0)
- moved TP10 131.9 mm to (231.5, 57.5)
- moved TP4 125.9 mm to (216.0, 62.0)
- moved TP8 120.7 mm to (214.0, 91.0)
- moved TP1 118.6 mm to (209.0, 59.0)
- moved TP13 110.1 mm to (209.0, 53.0)
- moved TP6 108.5 mm to (202.0, 80.0)
- moved R8 98.8 mm to (196.1, 61.0)
- moved R9 98.7 mm to (196.1, 64.0)
- moved Q2 98.0 mm to (203.1, 62.5)
- moved TP9 96.0 mm to (195.1, 68.0)
- moved TP7 95.6 mm to (190.0, 55.0)
- moved SW1 55.7 mm to (191.1, 62.0), turned to 180 degrees
- moved H1 39.0 mm to (183.0, 53.0)
- moved H4 39.0 mm to (183.0, 97.0)
- moved J3 31.9 mm to (184.0, 83.5), turned to 90 degrees
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Routing:
- net /VBAT: track 0.00 -> 94.6 mm, vias 0 -> 2
- net +3V3: track 0.00 -> 87.7 mm, vias 0 -> 4
- net /VBUS: track 0.00 -> 75.2 mm, vias 0 -> 2
- net +5V: track 0.00 -> 57.4 mm
- net /BTN_PWR: track 0.00 -> 28.8 mm, vias 0 -> 1
- net Net-(IC3-GND): track 0.00 -> 23.8 mm
- net Net-(IC2-~{STDBY}): track 0.00 -> 17.8 mm, vias 0 -> 2
- net GND: track 0.00 -> 17.5 mm
- net Net-(IC2-~{CHRG}): track 0.00 -> 16.9 mm, vias 0 -> 2
- net /PWR_HOLD: track 0.00 -> 14.7 mm
- net Net-(D3-A): track 0.00 -> 12.4 mm
- net Net-(IC3-VCC): track 0.00 -> 11.0 mm, vias 0 -> 2
- net Net-(IC3-OD): track 0.00 -> 10.7 mm
- net Net-(IC3-OC): track 0.00 -> 7.49 mm
- net Net-(IC1-FB): track 0.00 -> 6.74 mm
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- added copper zone on B.Cu, net GND
- added copper zone on F.Cu, net GND
Other:
- board size 100 x 50 mm -> 61 x 50 mm

Commit message: Power Board FREV2
Routing:
- net /VBAT: track 94.6 -> 110.4 mm
- net GND: vias 0 -> 33
