File: powerBoard/powerBoard.kicad_sch (KiCad schematic)
At the start: 43 parts, among them IC1 MT3608, IC2 TP4056, IC3 DW01A-G, J1 DATA, J2 PWR, J3 AUX, Q1 FS8205A, Q2 AO3401A, SW1 SW_SPST, U1 BAT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

Commit message: aa
Parts:
- added TP11, TP12: TestPoint, TestPoint:TestPoint_Pad_4.0x4.0mm, symbol Connector:TestPoint
- IC1: footprint SOT95P280X145-6N -> ChessLab:SOT95P280X145-6N
- IC2: footprint chessLab-footprints:SOIC127P600X175-9N -> ChessLab:SOIC127P600X175-9N
- IC3: footprint chessLab-footprints:SOT95P280X135-6N -> ChessLab:SOT95P280X135-6N
- L1: footprint chessLab-footprints:CDRH4D28NP100NC -> ChessLab:CDRH4D28NP100NC
- Q1: footprint chessLab-footprints:SOP65P640X120-8N -> ChessLab:SOP65P640X120-8N
- SW1: footprint chessLab-footprints:B3U-1000P -> ChessLab:B3U-1000P
- U1: footprint chessLab-footprints:CONN4_1048_KEY -> ChessLab:CONN4_1048_KEY
Changed lines of the file:
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@@
 			)
 		)
-		(property "Footprint" "chessLab-footprints:CONN4_1048_KEY"
+		(property "Footprint" "ChessLab:CONN4_1048_KEY"
 			(at 20.32 0.33 0)
 			(effects
@@
 			)
 		)
-		(property "Footprint" "chessLab-footprints:SOT95P280X135-6N"
+		(property "Footprint" "ChessLab:SOT95P280X135-6N"
 			(at 100.33 188.9 0)
 			(effects
@@
 			)
 		)
-		(property "Footprint" "chessLab-footprints:SOIC127P600X175-9N"
+		(property "Footprint" "ChessLab:SOIC127P600X175-9N"
 			(at 82.55 131.75 0)
 			(effects
@@
 	)
 	(symbol
+		(lib_id "Connector:TestPoint")
+		(at 25.4 113.03 0)
+		(unit 1)
+		(exclude_from_sim no)
+		(in_bom yes)
+		(on_board yes)
+		(dnp no)
+		(fields_autoplaced yes)
+		(property "Reference" "TP11"
+			(at 27.94 108.4579 0)
+			(effects
+				(font
+					(size 1.27 1.27)
+				)
+				(justify left)
+			)
+		)
+		(property "Value" "TestPoint"
+			(at 27.94 110.9979 0)
+			(effects
+				(font
+					(size 1.27 1.27)
+				)
+				(justify left)
+			)
+		)
+		(property "Footprint" "TestPoint:TestPoint_Pad_4.0x4.0mm"
+			(at 30.48 113.03 0)
+			(effects
+				(font
+					(size 1.27 1.27)
+				)
+				(hide yes)
+			)
+		)
+		(property "Datasheet" "~"
+			(at 30.48 113.03 0)
+			(effects
+				(font
+					(size 1.27 1.27)
+				)
+				(hide yes)
+			)
+		)
+		(property "Description" "test point"
+			(at 25.4 113.03 0)
+			(effects
+				(font
+					(size 1.27 1.27)
+				)
+				(hide yes)
+			)
+		)
+		(pin "1"
+		)
+		(instances
+			(project ""
+				(path "/ef9a6e1c-7dcb-475c-bb8f-502c132c52b8"
+					(reference "TP11")
+					(unit 1)
+				)
+			)
+		)
+	)
+	(symbol
 		(lib_id "Device:R")
 		(at 82.55 184.15 0)
@@
 			)
 		)
-		(property "Footprint" "chessLab-footprints:SOP65P640X120-8N"
+		(property "Footprint" "ChessLab:SOP65P640X120-8N"
 			(at 102.87 214.3 0)
 			(effects
@@
 			)
 		)
-		(property "Footprint" "SOT95P280X145-6N"
+		(property "Footprint" "ChessLab:SOT95P280X145-6N"
 			(at 64.77 263.83 0)
 			(effects
@@
 			)
 		)
-		(property "Footprint" "chessLab-footprints:CDRH4D28NP100NC"
+		(property "Footprint" "ChessLab:CDRH4D28NP100NC"
 			(at 148.26 142.24 0)
 			(effects
@@
 			)
 		)
-		(property "Footprint" "chessLab-footprints:B3U-1000P"
+		(property "Footprint" "ChessLab:B3U-1000P"
 			(at 160.02 105.41 0)
 			(effects
@@
 					(unit 1)
 				)
+			)
+		)
+	)
+	(symbol
+		(lib_id "Connector:TestPoint")
+		(at 39.37 113.03 0)
+		(unit 1)
+		(exclude_from_sim no)
+		(in_bom yes)
+		(on_board yes)
+		(dnp no)
+		(fields_autoplaced yes)
+		(property "Reference" "TP12"
+			(at 41.91 108.4579 0)
+			(effects
+				(font
+					(size 1.27 1.27)
+				)
+				(justify left)
+			)
+		)
+		(property "Value" "TestPoint"
+			(at 41.91 110.9979 0)
+			(effects
+				(font
+					(size 1.27 1.27)
+				)
+				(justify left)
+			)
+		)
+		(property "Footprint" "TestPoint:TestPoint_Pad_4.0x4.0mm"
+			(at 44.45 113.03 0)
+			(effects
+				(font
+					(size 1.27 1.27)
+				)
+				(hide yes)
+			)
+		)
+		(property "Datasheet" "~"
+			(at 44.45 113.03 0)
+			(effects
+				(font
+					(size 1.27 1.27)
+				)
+				(hide yes)
+			)
+		)
+		(property "Description" "test point"
+			(at 39.37 113.03 0)
+			(effects
+				(font
+					(size 1.27 1.27)
+				)
+				(hide yes)
+			)
+		)
+		(pin "1"
+		)
+		(instances
+			(project "powerBoard"
+				(path "/ef9a6e1c-7dcb-475c-bb8f-502c132c52b8"
+					(reference "TP12")
+					(unit 1)
+				)

Commit message: power pcb
Parts:
- removed TP2: +BAT, TestPoint:TestPoint_Plated_Hole_D2.0mm, symbol Connector:TestPoint
- removed U1: BAT, ChessLab:CONN4_1048_KEY, symbol chessLab-symbols:1048
- added H1, H2, H3, H4: MountingHole, MountingHole:MountingHole_2.7mm_M2.5, symbol Mechanical:MountingHole
- BAT+1: renamed from TP11; value TestPoint -> BAT+
- BAT-1: renamed from TP12; value TestPoint -> BAT-
- TP1, TP10, TP13, TP3, TP4, TP5, TP6, TP7, TP8, TP9: footprint TestPoint:TestPoint_Plated_Hole_D2.0mm -> TestPoint:TestPoint_Pad_D2.0mm
Connections:
- net VSYS is gone; now on net VBAT: C1.1, C6.1, IC1.4 (EN), IC1.5 (VIN), L1.1, Q2.3 (D), TP8.1, U2.3 (VI)
- net VBAT: now also BAT+1.1, R3.1
- net at C3.2, IC3.6 (GND), Q1.2 (S1_1)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: now also BAT-1.1
Other:
- moved on the sheet: BAT+1, BAT-1, TP5

Commit message: Power Board FREV2
Parts:
- removed R82: 0, Resistor_SMD:R_0603_1608Metric_Pad0.98x0.95mm_HandSolder, symbol Device:R
- removed TP3: GND, TestPoint:TestPoint_Pad_D2.0mm, symbol Connector:TestPoint
- removed TP5: VBAT, TestPoint:TestPoint_Pad_D2.0mm, symbol Connector:TestPoint
- added JP1: SolderJumper_2_Bridged, Jumper:SolderJumper-2_P1.3mm_Bridged2Bar_Pad1.0x1.5mm, symbol Jumper:SolderJumper_2_Bridged
Connections:
- net BTN_PWR: now also JP1.1 (A)
- net GND: now also JP1.2 (B)
Changed lines of the file:
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@@
 	)
 	(junction
-		(at 99.06 36.83)
-		(diameter 0)
-		(color 0 0 0 0)
-	)
-	(junction
 		(at 82.55 175.26)
 		(diameter 0)
@@
 	)
 	(junction
-		(at 71.12 64.77)
-		(diameter 0)
-		(color 0 0 0 0)
-	)
-	(junction
 		(at 170.18 33.02)
 		(diameter 0)
@@
 	(wire
 		(pts
-			(xy 91.44 36.83) (xy 99.06 36.83)
-		)
-		(stroke
-			(width 0)
-			(type default)
-		)
-	)
-	(wire
-		(pts
-			(xy 99.06 36.83) (xy 107.95 36.83)
+			(xy 91.44 36.83) (xy 107.95 36.83)
 		)
 		(stroke
@@
 	(wire
 		(pts
-			(xy 71.12 60.96) (xy 71.12 64.77)
+			(xy 71.12 60.96) (xy 71.12 67.31)
 		)
 		(stroke
@@
 	(wire
 		(pts
-			(xy 71.12 64.77) (xy 71.12 67.31)
-		)
-		(stroke
-			(width 0)
-			(type default)
-		)
-	)
-	(wire
-		(pts
 			(xy 71.12 57.15) (xy 71.12 60.96)
 		)
@@
 	(symbol
 		(lib_id "Device:R")
-		(at 161.29 175.26 90)
-		(unit 1)
-		(exclude_from_sim no)
-		(in_bom yes)
-		(on_board yes)
-		(dnp no)
-		(fields_autoplaced yes)
-		(property "Reference" "R82"
-			(at 161.29 168.91 90)
-			(effects
-				(font
-					(size 1.27 1.27)
-				)
-			)
-		)
-		(property "Value" "0"
-			(at 161.29 171.45 90)
-			(effects
-				(font
-					(size 1.27 1.27)
-				)
-			)
-		)
-		(property "Footprint" "Resistor_SMD:R_0603_1608Metric_Pad0.98x0.95mm_HandSolder"
-			(at 161.29 177.038 90)
-			(effects
-				(font
-					(size 1.27 1.27)
-				)
-				(hide yes)
-			)
-		)
-		(property "Datasheet" "~"
-			(at 161.29 175.26 0)
-			(effects
-				(font
-					(size 1.27 1.27)
-				)
-				(hide yes)
-			)
-		)
-		(property "Description" "Resistor"
-			(at 161.29 175.26 0)
-			(effects
-				(font
-					(size 1.27 1.27)
-				)
-				(hide yes)
-			)
-		)
-		(pin "2"
-		)
-		(pin "1"
-		)
-		(instances
-			(project "powerBoard"
-				(path "/ef9a6e1c-7dcb-475c-bb8f-502c132c52b8"
-					(reference "R82")
-					(unit 1)
-				)
-			)
-		)
-	)
-	(symbol
-		(lib_id "Device:R")
 		(at 35.56 48.26 0)
 		(unit 1)
@@
 	)
 	(symbol
-		(lib_id "Connector:TestPoint")
-		(at 71.12 64.77 90)
-		(unit 1)
-		(exclude_from_sim no)
-		(in_bom yes)
-		(on_board yes)
-		(dnp no)
-		(property "Reference" "TP3"
-			(at 64.516 65.786 0)
-			(effects
-				(font
-					(size 1.27 1.27)
-				)
-			)
-		)
-		(property "Value" "GND"
-			(at 62.484 66.04 0)
-			(effects
-				(font
-					(size 1.27 1.27)
-				)
-			)
-		)
-		(property "Footprint" "TestPoint:TestPoint_Pad_D2.0mm"
-			(at 71.12 59.69 0)
-			(effects
-				(font
-					(size 1.27 1.27)
-				)
-				(hide yes)
-			)
-		)
-		(property "Datasheet" "~"
-			(at 71.12 59.69 0)
-			(effects
-				(font
-					(size 1.27 1.27)
-				)
-				(hide yes)
-			)
-		)
-		(property "Description" "test point"
-			(at 71.12 64.77 0)
-			(effects
-				(font
-					(size 1.27 1.27)
-				)
-				(hide yes)
-			)
-		)
-		(pin "1"
-		)
-		(instances
-			(project "powerBoard"
-				(path "/ef9a6e1c-7dcb-475c-bb8f-502c132c52b8"
-					(reference "TP3")
-					(unit 1)
-				)
-			)
-		)
-	)
-	(symbol
 		(lib_id "chessLab-symbols:CDRH4D28NP-2R2NC")
 		(at 53.34 158.75 90)
@@
 	)
 	(symbol
-		(lib_id "Connector:TestPoint")
-		(at 99.06 36.83 180)
-		(unit 1)
-		(exclude_from_sim no)
-		(in_bom yes)
-		(on_board yes)
-		(dnp no)
-		(property "Reference" "TP5"
-			(at 100.076 43.434 0)
-			(effects
-				(font
-					(size 1.27 1.27)
-				)
-			)
-		)
-		(property "Value" "VBAT"
-			(at 100.33 45.466 0)
-			(effects
-				(font
-					(size 1.27 1.27)
-				)
-			)
-		)
-		(property "Footprint" "TestPoint:TestPoint_Pad_D2.0mm"
-			(at 93.98 36.83 0)
-			(effects
-				(font
-					(size 1.27 1.27)
-				)
-				(hide yes)
-			)
-		)
-		(property "Datasheet" "~"
-			(at 93.98 36.83 0)
-			(effects
-				(font
-					(size 1.27 1.27)
-				)
-				(hide yes)
-			)
-		)
-		(property "Description" "test point"
-			(at 99.06 36.83 0)
-			(effects
-				(font
-					(size 1.27 1.27)
-				)
-				(hide yes)
-			)
-		)
-		(pin "1"
-		)
-		(instances
-			(project "powerBoard"
-				(path "/ef9a6e1c-7dcb-475c-bb8f-502c132c52b8"
-					(reference "TP5")
-					(unit 1)
-				)
-			)
-		)
-	)
-	(symbol
 		(lib_id "Mechanical:MountingHole")
 		(at 217.335 121.5668 0)
@@
 					(unit 1)
 				)
+			)
+		)
+	)
+	(symbol
+		(lib_id "Jumper:SolderJumper_2_Bridged")
+		(at 161.29 175.26 0)
+		(unit 1)
+		(exclude_from_sim no)
+		(in_bom no)
+		(on_board yes)
+		(dnp no)
+		(fields_autoplaced yes)
+		(property "Reference" "JP1"
+			(at 161.29 168.91 0)
+			(effects
+				(font
+					(size 1.27 1.27)
+				)
+			)
+		)
+		(property "Value" "SolderJumper_2_Bridged"
+			(at 161.29 171.45 0)
+			(effects
+				(font
+					(size 1.27 1.27)
+				)
+				(hide yes)
+			)
+		)
+		(property "Footprint" "Jumper:SolderJumper-2_P1.3mm_Bridged2Bar_Pad1.0x1.5mm"
+			(at 161.29 175.26 0)
+			(effects
+				(font
+					(size 1.27 1.27)
+				)
+				(hide yes)
+			)
+		)
+		(property "Datasheet" "~"
+			(at 161.29 175.26 0)
+			(effects
+				(font
+					(size 1.27 1.27)
+				)
+				(hide yes)
+			)
+		)
+		(property "Description" "Solder Jumper, 2-pole, closed/bridged"
+			(at 161.29 175.26 0)
+			(effects
+				(font
+					(size 1.27 1.27)
+				)
+				(hide yes)
+			)
+		)
+		(pin "2"
+		)
+		(pin "1"
+		)
+		(instances
+			(project ""
+				(path "/ef9a6e1c-7dcb-475c-bb8f-502c132c52b8"
+					(reference "JP1")
+					(unit 1)
+				)
