File: Hardware/powerBoard/powerBoard.kicad_sch (KiCad schematic)
At the start: 44 parts, among them J4 DATA, J5 PWR, J6 AUX, Q1 FS8205A, Q2 AO3400A, U2 AMS1117-3.3, U3 DW01A, U4 MT3608, U5 TP4056

Commit message: ajout des vias et le nom sur la carte
Parts:
- D4, D5: footprint LED_SMD:LED_0603_1608Metric_Pad1.05x0.95mm_HandSolder -> LED_SMD:LED_0201_0603Metric
Changed lines of the file:
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@@
 			)
 		)
-		(property "Footprint" "LED_SMD:LED_0603_1608Metric_Pad1.05x0.95mm_HandSolder"
+		(property "Footprint" "LED_SMD:LED_0201_0603Metric"
 			(at 40.64 43.18 0)
 			(hide yes)
@@
 			)
 		)
-		(property "Footprint" "LED_SMD:LED_0603_1608Metric_Pad1.05x0.95mm_HandSolder"
+		(property "Footprint" "LED_SMD:LED_0201_0603Metric"
 			(at 29.21 50.8 0)
 			(hide yes)

Commit message: hist
Parts:
- D4, D5: footprint LED_SMD:LED_0201_0603Metric -> LED_SMD:LED_0603_1608Metric_Pad1.05x0.95mm_HandSolder
Changed lines of the file:
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@@
 			)
 		)
-		(property "Footprint" "LED_SMD:LED_0201_0603Metric"
+		(property "Footprint" "LED_SMD:LED_0603_1608Metric_Pad1.05x0.95mm_HandSolder"
 			(at 40.64 43.18 0)
 			(hide yes)
@@
 			)
 		)
-		(property "Footprint" "LED_SMD:LED_0201_0603Metric"
+		(property "Footprint" "LED_SMD:LED_0603_1608Metric_Pad1.05x0.95mm_HandSolder"
 			(at 29.21 50.8 0)
 			(hide yes)
