File: Hardware/powerBoard/powerBoard.kicad_pcb (KiCad board)
At the start: 2 copper layers, 56.1 x 37 mm, 44 parts, among them J4 DATA, J5 PWR, J6 AUX, Q1 FS8205A, Q2 AO3400A, U2 AMS1117-3.3, U3 DW01A, U4 MT3608, U5 TP4056

Commit message: ajout de via et les noms sur la carte
Routing:
- net GND: track 493.0 -> 493.7 mm, vias 142 -> 103
- net /VSYS: vias 3 -> 2
Other:
- board text added: "3V3"
- board text added: "5V"
- board text added: "BTN_PWR"
- board text added: "CONNECTE"
- board text added: "GND"
- board text added: "MAMADOU MOUCTAR BA ALEXANDRU CARP"
- board text added: "NON"
- board text added: "PWR_HOLD"
- board text added: "VBAT"
- board text added: "VBUS"
- board text removed: "MAMADOU MOUCTAR BA ET ALEXANDRU CARP"
